File: v2.0/main/com.kicad_sch (KiCad schematic)
At the start: 4 parts, among them J8 Conn_ARM_JTAG_SWD_10

Commit message: feat: update pcb routing
Parts:
- renumbered R32 to R30, R33 to R31, R34 to R32
Changed lines of the file:
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@@
 		(on_board yes)
 		(dnp no)
-		(property "Reference" "R33"
+		(property "Reference" "R31"
 			(at 124.46 83.82 0)
 			(effects
@@
 			(project ""
 				(path "/eb904614-38ff-4497-bc19-593801afccc5/773c3ee2-8fe5-42c9-964a-9e704f10744b"
-					(reference "R33")
+					(reference "R31")
 					(unit 1)
 				)
@@
 		(on_board yes)
 		(dnp no)
-		(property "Reference" "#PWR070"
+		(property "Reference" "#PWR063"
 			(at 123.19 83.82 0)
 			(effects
@@
 			(project ""
 				(path "/eb904614-38ff-4497-bc19-593801afccc5/773c3ee2-8fe5-42c9-964a-9e704f10744b"
-					(reference "#PWR070")
+					(reference "#PWR063")
 					(unit 1)
 				)
@@
 		(on_board yes)
 		(dnp no)
-		(property "Reference" "R32"
+		(property "Reference" "R30"
 			(at 118.11 83.82 0)
 			(effects
@@
 			(project ""
 				(path "/eb904614-38ff-4497-bc19-593801afccc5/773c3ee2-8fe5-42c9-964a-9e704f10744b"
-					(reference "R32")
+					(reference "R30")
 					(unit 1)
 				)
@@
 		(on_board yes)
 		(dnp no)
-		(property "Reference" "R34"
+		(property "Reference" "R32"
 			(at 130.81 83.82 0)
 			(effects
@@
 			(project ""
 				(path "/eb904614-38ff-4497-bc19-593801afccc5/773c3ee2-8fe5-42c9-964a-9e704f10744b"
-					(reference "R34")
+					(reference "R32")
 					(unit 1)
 				)
@@
 				)
 				(justify right)
+				(hide yes)
 			)
 		)
@@
 		(on_board yes)
 		(dnp no)
-		(property "Reference" "#PWR069"
+		(property "Reference" "#PWR062"
 			(at 105.41 120.65 0)
 			(effects
@@
 			(project ""
 				(path "/eb904614-38ff-4497-bc19-593801afccc5/773c3ee2-8fe5-42c9-964a-9e704f10744b"
-					(reference "#PWR069")
+					(reference "#PWR062")
 					(unit 1)
 				)
@@
 		(on_board yes)
 		(dnp no)
-		(property "Reference" "#PWR068"
+		(property "Reference" "#PWR061"
 			(at 105.41 83.82 0)
 			(effects
@@
 			(project ""
 				(path "/eb904614-38ff-4497-bc19-593801afccc5/773c3ee2-8fe5-42c9-964a-9e704f10744b"
-					(reference "#PWR068")
-					(unit 1)
-				)
+					(reference "#PWR061")
+					(unit 1)
+				)
