File: v2.0/main/fan_motor.kicad_sch (KiCad schematic)
At the start: 4 parts, among them J9 Conn_01x02, Q9 IRFML8244

Commit message: feat: update pcb routing
Parts:
- J9: footprint Connector_PinSocket_1.27mm:PinSocket_1x02_P1.27mm_Vertical -> Connector_PinHeader_1.00mm:PinHeader_1x02_P1.00mm_Vertical
- renumbered Q9 to Q7, R35 to R33, R36 to R34
Changed lines of the file:
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@@
 		(on_board yes)
 		(dnp no)
-		(property "Reference" "R35"
+		(property "Reference" "R33"
 			(at 121.92 100.4316 90)
 			(effects
@@
 			(project "main"
 				(path "/eb904614-38ff-4497-bc19-593801afccc5/4a74c57e-dfd6-4d81-99fe-e893bb89d00d"
-					(reference "R35")
+					(reference "R33")
 					(unit 1)
 				)
@@
 		(on_board yes)
 		(dnp no)
-		(property "Reference" "#PWR072"
+		(property "Reference" "#PWR065"
 			(at 135.89 130.81 0)
 			(effects
@@
 			(project "main"
 				(path "/eb904614-38ff-4497-bc19-593801afccc5/4a74c57e-dfd6-4d81-99fe-e893bb89d00d"
-					(reference "#PWR072")
+					(reference "#PWR065")
 					(unit 1)
 				)
@@
 		(on_board yes)
 		(dnp no)
-		(property "Reference" "Q9"
+		(property "Reference" "Q7"
 			(at 138.557 104.2416 0)
 			(effects
@@
 			(project "main"
 				(path "/eb904614-38ff-4497-bc19-593801afccc5/4a74c57e-dfd6-4d81-99fe-e893bb89d00d"
-					(reference "Q9")
+					(reference "Q7")
 					(unit 1)
 				)
@@
 		(on_board yes)
 		(dnp no)
-		(property "Reference" "#PWR071"
+		(property "Reference" "#PWR064"
 			(at 135.89 83.82 0)
 			(effects
@@
 			(project "main"
 				(path "/eb904614-38ff-4497-bc19-593801afccc5/4a74c57e-dfd6-4d81-99fe-e893bb89d00d"
-					(reference "#PWR071")
+					(reference "#PWR064")
 					(unit 1)
 				)
@@
 			)
 		)
-		(property "Footprint" "Connector_PinSocket_1.27mm:PinSocket_1x02_P1.27mm_Vertical"
+		(property "Footprint" "Connector_PinHeader_1.00mm:PinHeader_1x02_P1.00mm_Vertical"
 			(at 140.97 88.9 0)
 			(effects
@@
 		(on_board yes)
 		(dnp no)
-		(property "Reference" "R36"
+		(property "Reference" "R34"
 			(at 128.4986 111.8616 0)
 			(effects
@@
 			(project "main"
 				(path "/eb904614-38ff-4497-bc19-593801afccc5/4a74c57e-dfd6-4d81-99fe-e893bb89d00d"
-					(reference "R36")
-					(unit 1)
-				)
+					(reference "R34")
+					(unit 1)
+				)
