File: v2.0/main/ir_led.kicad_sch (KiCad schematic)
At the start: 6 parts, among them Q7 PMF250XNEX

Commit message: feat: update pcb routing
Parts:
- renumbered D10 to D12, D11 to D13
Changed lines of the file:
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@@
 		(dnp no)
 		(fields_autoplaced yes)
-		(property "Reference" "#PWR065"
+		(property "Reference" "#PWR062"
 			(at 137.16 130.81 0)
 			(effects
@@
 			(project ""
 				(path "/eb904614-38ff-4497-bc19-593801afccc5/20720b4c-26bd-4017-891c-b78b41525f4b"
-					(reference "#PWR065")
-					(unit 1)
-				)
-				(path "/eb904614-38ff-4497-bc19-593801afccc5/d5650c90-80e2-4a62-9769-29a8f78adcb5"
-					(reference "#PWR067")
+					(reference "#PWR062")
+					(unit 1)
+				)
+				(path "/eb904614-38ff-4497-bc19-593801afccc5/d5650c90-80e2-4a62-9769-29a8f78adcb5"
+					(reference "#PWR064")
 					(unit 1)
 				)
@@
 		(dnp no)
 		(fields_autoplaced yes)
-		(property "Reference" "D10"
+		(property "Reference" "D12"
 			(at 140.97 82.8674 90)
 			(effects
@@
 			(project ""
 				(path "/eb904614-38ff-4497-bc19-593801afccc5/20720b4c-26bd-4017-891c-b78b41525f4b"
-					(reference "D10")
-					(unit 1)
-				)
-				(path "/eb904614-38ff-4497-bc19-593801afccc5/d5650c90-80e2-4a62-9769-29a8f78adcb5"
 					(reference "D12")
+					(unit 1)
+				)
+				(path "/eb904614-38ff-4497-bc19-593801afccc5/d5650c90-80e2-4a62-9769-29a8f78adcb5"
+					(reference "D14")
 					(unit 1)
 				)
@@
 		(dnp no)
 		(fields_autoplaced yes)
-		(property "Reference" "D11"
+		(property "Reference" "D13"
 			(at 140.97 90.4874 90)
 			(effects
@@
 			(project ""
 				(path "/eb904614-38ff-4497-bc19-593801afccc5/20720b4c-26bd-4017-891c-b78b41525f4b"
-					(reference "D11")
-					(unit 1)
-				)
-				(path "/eb904614-38ff-4497-bc19-593801afccc5/d5650c90-80e2-4a62-9769-29a8f78adcb5"
 					(reference "D13")
+					(unit 1)
+				)
+				(path "/eb904614-38ff-4497-bc19-593801afccc5/d5650c90-80e2-4a62-9769-29a8f78adcb5"
+					(reference "D15")
 					(unit 1)
 				)
@@
 		(dnp no)
 		(fields_autoplaced yes)
-		(property "Reference" "#PWR064"
+		(property "Reference" "#PWR061"
 			(at 140.97 76.2 0)
 			(effects
@@
 			(project ""
 				(path "/eb904614-38ff-4497-bc19-593801afccc5/20720b4c-26bd-4017-891c-b78b41525f4b"
-					(reference "#PWR064")
-					(unit 1)
-				)
-				(path "/eb904614-38ff-4497-bc19-593801afccc5/d5650c90-80e2-4a62-9769-29a8f78adcb5"
-					(reference "#PWR066")
-					(unit 1)
-				)
+					(reference "#PWR061")
+					(unit 1)
+				)
+				(path "/eb904614-38ff-4497-bc19-593801afccc5/d5650c90-80e2-4a62-9769-29a8f78adcb5"
+					(reference "#PWR063")
+					(unit 1)
+				)
