File: v2.0/main/ir_sensor.kicad_sch (KiCad schematic)
At the start: 2 parts, among them Q4 LTR-209

Commit message: feat: update pcb routing
Parts:
- removed R23: 1k, Resistor_SMD:R_0201_0603Metric, symbol Device:R_Small
- added C21: 0.1u, Capacitor_SMD:C_0402_1005Metric, symbol Device:C
- added R24: 1.5k, Resistor_SMD:R_0402_1005Metric, symbol Device:R
- added R25: 10k, Resistor_SMD:R_0402_1005Metric, symbol Device:R
- Q4: value LTR-209 -> OP505A; check_order (none) -> ok; order_URL (none) -> https://www.digikey.jp/ja/products/detail/tt-electronics-op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
Connections:
- net GND: now also R24.2, R25.2
- net IR_RCV: now also C21.1, R25.1; no longer Q4.2 (E)
- net +3.3VADC renamed +3.3V
- new net: C21.2, Q4.2 (E), R24.1
Other:
- note added: "3.3=V_{CE}+R*I_{C} R=(3.3-V_{CE})/I_{C} V_{CE}=0.4 [V] I_{C}=4.3 [mA] (3.3-0.4)/0.002=145 R=1.5 k"
- note added: "HPF for 50/60Hz Light fc=100~200 Hz R=10k C=0.1u fc=160 Hz"
