File: v2.0/main/main.kicad_sch (KiCad schematic)
At the start: 14 parts, among them SW1 TVAF06-A020B-R, U1 STM32F411CEUx, Y1 XRCGB16M000FXN02R0

Commit message: feat: update pcb routing
Parts:
- removed C1, C2: 10p, Capacitor_SMD:C_0402_1005Metric_Pad0.74x0.62mm_HandSolder, symbol Device:C_Small
- removed R1: 1k, Resistor_SMD:R_0402_1005Metric_Pad0.72x0.64mm_HandSolder, symbol Device:R_Small
- removed Y1: XRCGB16M000FXN02R0, bldc:XRCGB16M000FXN02R0, symbol Device:Crystal_GND2_Small
- added C8: 0.1u, Capacitor_SMD:C_0201_0603Metric, symbol Device:C_Small
- renumbered C3 to C1, C4 to C2, C5 to C3, C6 to C4, C7 to C5, C8 to C6, C9 to C7, R2 to R1
Connections:
- net +3.3VADC is gone; now on net +3.3V: U1.9 (VDDA)
- net OSC_IN is gone; now on net USER_LED10: U1.5 (PH0)
- net OSC_OUT is gone; now on net USER_SW: U1.6 (PH1)
- net +3.3V: now also C8.1
- net GND: now also C8.2
- net IR_LED_F: now also U1.19 (PB1); no longer U1.16 (PA6)
- net IR_LED_S: now also U1.16 (PA6); no longer U1.19 (PB1)
- net USER_LED1: now also U1.31 (PA10); no longer U1.20 (PB2)
- net USER_LED10: no longer U1.4 (PC15)
- net USER_LED2: now also U1.32 (PA11); no longer U1.21 (PB10)
- net USER_LED3: now also U1.33 (PA12); no longer U1.31 (PA10)
- net USER_LED4: now also U1.38 (PA15); no longer U1.32 (PA11)
- net USER_LED5: now also U1.39 (PB3); no longer U1.38 (PA15)
- net USER_LED6: now also U1.40 (PB4); no longer U1.39 (PB3)
- net USER_LED7: now also U1.2 (PC13); no longer U1.40 (PB4)
- net USER_LED8: now also U1.3 (PC14); no longer U1.2 (PC13)
- net USER_LED9: now also U1.4 (PC15); no longer U1.3 (PC14)
- net USER_SW: no longer U1.33 (PA12)
Other:
- removed sheet ir_led_F
- removed sheet ir_led_S
- added sheet wall_senso_S (wall_sensor.kicad_sch)
- added sheet wall_sensor_F (wall_sensor.kicad_sch)
