File: v2.0/main/encoder.kicad_sch (KiCad schematic)
At the start: 6 parts, among them J6 enc_host, J7 enc_slave, U6 MA730

Commit message: feat: update pcb routing
Parts:
- J6: footprint Connector_PinHeader_1.27mm:PinHeader_1x04_P1.27mm_Vertical -> half_mouse_lib:enc_fp
- J7: footprint (none) -> half_mouse_lib:enc_board
- renumbered C20 to C19, R11 to R10, R12 to R11
Connections:
- net ENC_A: now also J7.3 (Pin_3); no longer J7.2 (Pin_2)
- net ENC_B: now also J7.2 (Pin_2); no longer J7.3 (Pin_3)
Changed lines of the file:
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@@
 		)
 	)
-	(label "ENC_A"
+	(label "ENC_B"
 		(at 153.67 49.53 0)
 		(fields_autoplaced yes)
@@
 		)
 	)
-	(label "ENC_B"
+	(label "ENC_A"
 		(at 153.67 52.07 0)
 		(fields_autoplaced yes)
@@
 		(on_board yes)
 		(dnp no)
-		(property "Reference" "R12"
+		(property "Reference" "R11"
 			(at 139.7 97.79 0)
 			(effects
@@
 			(project "main"
 				(path "/eb904614-38ff-4497-bc19-593801afccc5/b149e7a9-a2a2-4697-b2ac-eb9ad11b51d2"
-					(reference "R12")
-					(unit 1)
-				)
-				(path "/eb904614-38ff-4497-bc19-593801afccc5/ddac4fdd-1c79-48b6-9f0c-f62653388747"
-					(reference "R4")
+					(reference "R11")
+					(unit 1)
+				)
+				(path "/eb904614-38ff-4497-bc19-593801afccc5/ddac4fdd-1c79-48b6-9f0c-f62653388747"
+					(reference "R3")
 					(unit 1)
 				)
@@
 		(dnp no)
 		(fields_autoplaced yes)
-		(property "Reference" "#PWR045"
+		(property "Reference" "#PWR040"
 			(at 101.6 63.5 0)
 			(effects
@@
 			(project "main"
 				(path "/eb904614-38ff-4497-bc19-593801afccc5/b149e7a9-a2a2-4697-b2ac-eb9ad11b51d2"
-					(reference "#PWR045")
-					(unit 1)
-				)
-				(path "/eb904614-38ff-4497-bc19-593801afccc5/ddac4fdd-1c79-48b6-9f0c-f62653388747"
-					(reference "#PWR011")
+					(reference "#PWR040")
+					(unit 1)
+				)
+				(path "/eb904614-38ff-4497-bc19-593801afccc5/ddac4fdd-1c79-48b6-9f0c-f62653388747"
+					(reference "#PWR09")
 					(unit 1)
 				)
@@
 		(dnp no)
 		(fields_autoplaced yes)
-		(property "Reference" "C20"
+		(property "Reference" "C19"
 			(at 99.06 77.4762 0)
 			(effects
@@
 			(project ""
 				(path "/eb904614-38ff-4497-bc19-593801afccc5/b149e7a9-a2a2-4697-b2ac-eb9ad11b51d2"
-					(reference "C20")
-					(unit 1)
-				)
-				(path "/eb904614-38ff-4497-bc19-593801afccc5/ddac4fdd-1c79-48b6-9f0c-f62653388747"
-					(reference "C10")
+					(reference "C19")
+					(unit 1)
+				)
+				(path "/eb904614-38ff-4497-bc19-593801afccc5/ddac4fdd-1c79-48b6-9f0c-f62653388747"
+					(reference "C9")
 					(unit 1)
 				)
@@
 		(on_board yes)
 		(dnp no)
-		(property "Reference" "R11"
+		(property "Reference" "R10"
 			(at 132.08 97.79 0)
 			(effects
@@
 			(project "main"
 				(path "/eb904614-38ff-4497-bc19-593801afccc5/b149e7a9-a2a2-4697-b2ac-eb9ad11b51d2"
-					(reference "R11")
-					(unit 1)
-				)
-				(path "/eb904614-38ff-4497-bc19-593801afccc5/ddac4fdd-1c79-48b6-9f0c-f62653388747"
-					(reference "R3")
+					(reference "R10")
+					(unit 1)
+				)
+				(path "/eb904614-38ff-4497-bc19-593801afccc5/ddac4fdd-1c79-48b6-9f0c-f62653388747"
+					(reference "R2")
 					(unit 1)
 				)
@@
 			)
 		)
-		(property "Footprint" "Connector_PinHeader_1.27mm:PinHeader_1x04_P1.27mm_Vertical"
+		(property "Footprint" "half_mouse_lib:enc_fp"
 			(at 109.22 49.53 0)
 			(effects
@@
 		(dnp no)
 		(fields_autoplaced yes)
-		(property "Reference" "#PWR044"
+		(property "Reference" "#PWR039"
 			(at 101.6 48.26 0)
 			(effects
@@
 			(project "main"
 				(path "/eb904614-38ff-4497-bc19-593801afccc5/b149e7a9-a2a2-4697-b2ac-eb9ad11b51d2"
-					(reference "#PWR044")
-					(unit 1)
-				)
-				(path "/eb904614-38ff-4497-bc19-593801afccc5/ddac4fdd-1c79-48b6-9f0c-f62653388747"
-					(reference "#PWR010")
+					(reference "#PWR039")
+					(unit 1)
+				)
+				(path "/eb904614-38ff-4497-bc19-593801afccc5/ddac4fdd-1c79-48b6-9f0c-f62653388747"
+					(reference "#PWR08")
 					(unit 1)
 				)
@@
 			)
 		)
-		(property "Footprint" ""
+		(property "Footprint" "half_mouse_lib:enc_board"
 			(at 142.24 49.53 0)
 			(effects

Commit message: fix: parts position
Connections:
- net ENC_A: now also J6.3 (Pin_3); no longer J6.2 (Pin_2), J7.3 (Pin_3), U6.2 (A)
- net ENC_B: now also J6.2 (Pin_2); no longer J6.3 (Pin_3), J7.2 (Pin_2), U6.6 (B)
- net s_GND: now also J7.1 (Pin_1); no longer J7.4 (Pin_4)
- net s_VDD: now also J7.4 (Pin_4); no longer J7.1 (Pin_1)
- new net ENC_A_: J7.2 (Pin_2), U6.2 (A)
- new net ENC_B_: J7.3 (Pin_3), U6.6 (B)
Changed lines of the file:
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@@
+	)
+	(junction
+		(at 149.86 46.99)
+		(diameter 0)
+		(color 0 0 0 0)
 	)
 	(junction
@@
 	)
 	(junction
-		(at 149.86 46.99)
-		(diameter 0)
-		(color 0 0 0 0)
-	)
-	(junction
 		(at 106.68 74.93)
 		(diameter 0)
@@
 	(wire
 		(pts
+			(xy 147.32 46.99) (xy 149.86 46.99)
+		)
+		(stroke
+			(width 0)
+			(type default)
+		)
+	)
+	(wire
+		(pts
 			(xy 149.86 44.45) (xy 149.86 46.99)
 		)
@@
 	(wire
 		(pts
-			(xy 147.32 46.99) (xy 149.86 46.99)
+			(xy 147.32 54.61) (xy 149.86 54.61)
 		)
 		(stroke
@@
 	(wire
 		(pts
+			(xy 137.16 92.71) (xy 137.16 96.52)
+		)
+		(stroke
+			(width 0)
+			(type default)
+		)
+	)
+	(wire
+		(pts
+			(xy 119.38 92.71) (xy 137.16 92.71)
+		)
+		(stroke
+			(width 0)
+			(type default)
+		)
+	)
+	(wire
+		(pts
+			(xy 121.92 97.79) (xy 119.38 97.79)
+		)
+		(stroke
+			(width 0)
+			(type default)
+		)
+	)
+	(wire
+		(pts
+			(xy 101.6 52.07) (xy 104.14 52.07)
+		)
+		(stroke
+			(width 0)
+			(type default)
+		)
+	)
+	(wire
+		(pts
+			(xy 144.78 101.6) (xy 144.78 106.68)
+		)
+		(stroke
+			(width 0)
+			(type default)
+		)
+	)
+	(wire
+		(pts
+			(xy 106.68 74.93) (xy 106.68 82.55)
+		)
+		(stroke
+			(width 0)
+			(type default)
+		)
+	)
+	(wire
+		(pts
+			(xy 104.14 113.03) (xy 106.68 113.03)
+		)
+		(stroke
+			(width 0)
+			(type default)
+		)
+	)
+	(wire
+		(pts
 			(xy 147.32 49.53) (xy 153.67 49.53)
 		)
@@
 	(wire
 		(pts
-			(xy 137.16 92.71) (xy 137.16 96.52)
-		)
-		(stroke
-			(width 0)
-			(type default)
-		)
-	)
-	(wire
-		(pts
-			(xy 119.38 92.71) (xy 137.16 92.71)
-		)
-		(stroke
-			(width 0)
-			(type default)
-		)
-	)
-	(wire
-		(pts
-			(xy 121.92 97.79) (xy 119.38 97.79)
-		)
-		(stroke
-			(width 0)
-			(type default)
-		)
-	)
-	(wire
-		(pts
-			(xy 101.6 52.07) (xy 104.14 52.07)
-		)
-		(stroke
-			(width 0)
-			(type default)
-		)
-	)
-	(wire
-		(pts
-			(xy 144.78 101.6) (xy 144.78 106.68)
-		)
-		(stroke
-			(width 0)
-			(type default)
-		)
-	)
-	(wire
-		(pts
-			(xy 106.68 74.93) (xy 106.68 82.55)
-		)
-		(stroke
-			(width 0)
-			(type default)
-		)
-	)
-	(wire
-		(pts
-			(xy 104.14 113.03) (xy 106.68 113.03)
-		)
-		(stroke
-			(width 0)
-			(type default)
-		)
-	)
-	(wire
-		(pts
 			(xy 144.78 90.17) (xy 144.78 96.52)
 		)
@@
 		(pts
 			(xy 96.52 74.93) (xy 106.68 74.93)
-		)
-		(stroke
-			(width 0)
-			(type default)
-		)
-	)
-	(wire
-		(pts
-			(xy 149.86 54.61) (xy 147.32 54.61)
 		)
 		(stroke
@@
 		)
 	)
-	(label "ENC_B"
+	(label "ENC_B_"
 		(at 121.92 100.33 0)
 		(fields_autoplaced yes)
@@
 		)
 	)
-	(label "ENC_B"
+	(label "ENC_B_"
 		(at 153.67 49.53 0)
 		(fields_autoplaced yes)
@@
 		)
 	)
-	(label "ENC_A"
+	(label "ENC_A_"
 		(at 121.92 97.79 0)
 		(fields_autoplaced yes)
@@
 		)
 	)
-	(label "ENC_A"
+	(label "ENC_A_"
 		(at 153.67 52.07 0)
 		(fields_autoplaced yes)
@@
 		)
 	)
-	(hierarchical_label "ENC_B"
+	(hierarchical_label "ENC_A"
 		(shape input)
 		(at 101.6 52.07 180)
@@
 		)
 	)
-	(hierarchical_label "ENC_A"
+	(hierarchical_label "ENC_B"
 		(shape input)
 		(at 101.6 49.53 180)
@@
 	(symbol
 		(lib_id "Connector:Conn_01x04_Pin")
-		(at 142.24 49.53 0)
+		(at 142.24 52.07 0)
+		(mirror x)
 		(unit 1)
 		(exclude_from_sim no)
@@
 		(dnp no)
 		(property "Reference" "J7"
+			(at 136.652 52.07 0)
+			(effects
+				(font
+					(size 1.27 1.27)
+				)
+			)
+		)
+		(property "Value" "enc_slave"
 			(at 136.652 49.53 0)
 			(effects
@@
 			)
 		)
-		(property "Value" "enc_slave"
-			(at 136.652 52.07 0)
-			(effects
-				(font
-					(size 1.27 1.27)
-				)
-			)
-		)
 		(property "Footprint" "half_mouse_lib:enc_board"
-			(at 142.24 49.53 0)
+			(at 142.24 52.07 0)
 			(effects
 				(font
@@
 		)
 		(property "Datasheet" "~"
-			(at 142.24 49.53 0)
+			(at 142.24 52.07 0)
 			(effects
 				(font
@@
 		)
 		(property "Description" "Generic connector, single row, 01x04, script generated"
-			(at 142.24 49.53 0)
-			(effects
-				(font
+			(at 142.24 52.07 0)
+			(effects
+				(font

Commit message: feat: order to JLCPCB
Parts:
- C19: value 1u -> 0.1u
Changed lines of the file:
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@@
 			)
 		)
-		(property "Value" "1u"
+		(property "Value" "0.1u"
 			(at 99.06 80.0162 0)
 			(effects
