File: v2.0/main/motor.kicad_sch (KiCad schematic)
At the start: 8 parts, among them J3 motor_L, J4 motor_R, U4 DRV8835

Commit message: feat: update pcb routing
Parts:
- C15: renamed from C16; footprint Capacitor_SMD:C_0603_1608Metric -> Capacitor_SMD:C_0402_1005Metric
- J3, J4: footprint half_mouse_lib:motor_SMD -> Connector_PinHeader_1.00mm:PinHeader_1x02_P1.00mm_Vertical
- renumbered C14 to C13, C15 to C14
Connections:
- net at L2.1: now also U4.4 (BOUT1); no longer U4.5 (BOUT2)
- net at L2.2: now also J4.1 (Pin_1); no longer J4.2 (Pin_2)
- new net: J4.2 (Pin_2), U4.5 (BOUT2)
Other:
- moved on the sheet: L2
Changed lines of the file:
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@@
+	(wire
+		(pts
+			(xy 144.78 87.63) (xy 147.32 87.63)
+		)
+		(stroke
+			(width 0)
+			(type default)
+		)
+	)
 	(wire
 		(pts
@@
 	(wire
 		(pts
-			(xy 144.78 87.63) (xy 156.21 87.63)
-		)
-		(stroke
-			(width 0)
-			(type default)
-		)
-	)
-	(wire
-		(pts
 			(xy 113.03 82.55) (xy 118.11 82.55)
 		)
@@
 	(wire
 		(pts
-			(xy 144.78 90.17) (xy 147.32 90.17)
+			(xy 154.94 87.63) (xy 156.21 87.63)
 		)
 		(stroke
@@
 	(wire
 		(pts
-			(xy 154.94 90.17) (xy 156.21 90.17)
-		)
-		(stroke
-			(width 0)
-			(type default)
-		)
-	)
-	(wire
-		(pts
 			(xy 60.96 77.47) (xy 60.96 87.63)
 		)
@@
 		(pts
 			(xy 82.55 100.33) (xy 82.55 92.71)
+		)
+		(stroke
+			(width 0)
+			(type default)
+		)
+	)
+	(wire
+		(pts
+			(xy 144.78 90.17) (xy 156.21 90.17)
 		)
 		(stroke
@@
 		(on_board yes)
 		(dnp no)
-		(property "Reference" "C16"
+		(property "Reference" "C15"
 			(at 74.93 88.9 0)
 			(effects
@@
 			)
 		)
-		(property "Footprint" "Capacitor_SMD:C_0603_1608Metric"
+		(property "Footprint" "Capacitor_SMD:C_0402_1005Metric"
 			(at 82.55 90.17 0)
 			(effects
@@
 			(project ""
 				(path "/eb904614-38ff-4497-bc19-593801afccc5/1067b3be-65e2-4ccf-8892-c72fee81dea1"
-					(reference "C16")
+					(reference "C15")
 					(unit 1)
 				)
@@
 		(dnp no)
 		(fields_autoplaced yes)
-		(property "Reference" "#PWR026"
+		(property "Reference" "#PWR024"
 			(at 133.35 109.22 0)
 			(effects
@@
 			(project ""
 				(path "/eb904614-38ff-4497-bc19-593801afccc5/1067b3be-65e2-4ccf-8892-c72fee81dea1"
-					(reference "#PWR026")
+					(reference "#PWR024")
 					(unit 1)
 				)
@@
 	(symbol
 		(lib_id "Device:L")
-		(at 151.13 90.17 90)
+		(at 151.13 87.63 90)
 		(unit 1)
 		(exclude_from_sim no)
@@
 		(dnp no)
 		(property "Reference" "L2"
+			(at 151.13 90.17 90)
+			(effects
+				(font
+					(size 1.27 1.27)
+				)
+			)
+		)
+		(property "Value" "47u"
 			(at 151.13 92.71 90)
 			(effects
@@
 			)
 		)
-		(property "Value" "47u"
-			(at 151.13 95.25 90)
-			(effects
-				(font
-					(size 1.27 1.27)
-				)
-			)
-		)
 		(property "Footprint" "Inductor_SMD:L_0603_1608Metric_Pad1.05x0.95mm_HandSolder"
-			(at 151.13 90.17 0)
+			(at 151.13 87.63 0)
 			(effects
 				(font
@@
 		)
 		(property "Datasheet" "~"
-			(at 151.13 90.17 0)
-			(effects
-				(font
-					(size 1.27 1.27)
-				)
-				(hide yes)
-			)
-		)
-		(property "Description" ""
-			(at 151.13 90.17 0)
+			(at 151.13 87.63 0)
+			(effects
+				(font
+					(size 1.27 1.27)
+				)
+				(hide yes)
+			)
+		)
+		(property "Description" ""
+			(at 151.13 87.63 0)
 			(effects
 				(font
@@
 		(on_board yes)
 		(dnp no)
-		(property "Reference" "#PWR025"
+		(property "Reference" "#PWR023"
 			(at 133.35 80.01 0)
 			(effects
@@
 			(project ""
 				(path "/eb904614-38ff-4497-bc19-593801afccc5/1067b3be-65e2-4ccf-8892-c72fee81dea1"
-					(reference "#PWR025")
+					(reference "#PWR023")
 					(unit 1)
 				)
@@
 		(on_board yes)
 		(dnp no)
-		(property "Reference" "#PWR020"
+		(property "Reference" "#PWR018"
 			(at 72.39 81.28 0)
 			(effects
@@
 			(project ""
 				(path "/eb904614-38ff-4497-bc19-593801afccc5/1067b3be-65e2-4ccf-8892-c72fee81dea1"
-					(reference "#PWR020")
+					(reference "#PWR018")
 					(unit 1)
 				)
@@
 		(dnp no)
 		(fields_autoplaced yes)
-		(property "Reference" "#PWR019"
+		(property "Reference" "#PWR017"
 			(at 60.96 109.22 0)
 			(effects
@@
 			(project ""
 				(path "/eb904614-38ff-4497-bc19-593801afccc5/1067b3be-65e2-4ccf-8892-c72fee81dea1"
-					(reference "#PWR019")
+					(reference "#PWR017")
 					(unit 1)
 				)
@@
 		(on_board yes)
 		(dnp no)
-		(property "Reference" "C15"
+		(property "Reference" "C14"
 			(at 64.77 88.9 0)
 			(effects
@@
 			(project ""
 				(path "/eb904614-38ff-4497-bc19-593801afccc5/1067b3be-65e2-4ccf-8892-c72fee81dea1"
-					(reference "C15")
+					(reference "C14")
 					(unit 1)
 				)
@@
 			)
 		)
-		(property "Footprint" "half_mouse_lib:motor_SMD"
+		(property "Footprint" "Connector_PinHeader_1.00mm:PinHeader_1x02_P1.00mm_Vertical"
 			(at 161.29 87.63 0)
 			(effects
@@
 			)
 		)
-		(property "Footprint" "half_mouse_lib:motor_SMD"
+		(property "Footprint" "Connector_PinHeader_1.00mm:PinHeader_1x02_P1.00mm_Vertical"
 			(at 161.29 82.55 0)
 			(effects
@@
 		(dnp no)
 		(fields_autoplaced yes)
-		(property "Reference" "#PWR021"
+		(property "Reference" "#PWR019"
 			(at 72.39 109.22 0)
 			(effects
@@
 			(project ""
 				(path "/eb904614-38ff-4497-bc19-593801afccc5/1067b3be-65e2-4ccf-8892-c72fee81dea1"
-					(reference "#PWR021")
+					(reference "#PWR019")
 					(unit 1)
 				)
@@
 		(dnp no)
 		(fields_autoplaced yes)
-		(property "Reference" "#PWR023"
+		(property "Reference" "#PWR021"
 			(at 129.54 80.01 0)
 			(effects
@@
 			(project ""
 				(path "/eb904614-38ff-4497-bc19-593801afccc5/1067b3be-65e2-4ccf-8892-c72fee81dea1"
-					(reference "#PWR023")
+					(reference "#PWR021")
 					(unit 1)
 				)
@@
 		(dnp no)
 		(fields_autoplaced yes)
-		(property "Reference" "#PWR018"
+		(property "Reference" "#PWR016"
 			(at 60.96 81.28 0)
 			(effects
@@
 			(project ""
 				(path "/eb904614-38ff-4497-bc19-593801afccc5/1067b3be-65e2-4ccf-8892-c72fee81dea1"
-					(reference "#PWR018")
+					(reference "#PWR016")
 					(unit 1)
 				)
@@
 		(dnp no)
 		(fields_autoplaced yes)
-		(property "Reference" "#PWR022"
+		(property "Reference" "#PWR020"
 			(at 118.11 109.22 0)
 			(effects
@@
 			(project ""
 				(path "/eb904614-38ff-4497-bc19-593801afccc5/1067b3be-65e2-4ccf-8892-c72fee81dea1"
-					(reference "#PWR022")
+					(reference "#PWR020")
 					(unit 1)
 				)
@@
 		(on_board yes)
 		(dnp no)
-		(property "Reference" "C14"
+		(property "Reference" "C13"
 			(at 53.34 88.9 0)
 			(effects
@@
 			(project ""
 				(path "/eb904614-38ff-4497-bc19-593801afccc5/1067b3be-65e2-4ccf-8892-c72fee81dea1"
-					(reference "C14")
+					(reference "C13")
 					(unit 1)
 				)
@@
 		(dnp no)
 		(fields_autoplaced yes)
-		(property "Reference" "#PWR024"
+		(property "Reference" "#PWR022"
 			(at 129.54 109.22 0)
 			(effects
@@
 			(project ""
 				(path "/eb904614-38ff-4497-bc19-593801afccc5/1067b3be-65e2-4ccf-8892-c72fee81dea1"
-					(reference "#PWR024")
-					(unit 1)
-				)
+					(reference "#PWR022")
+					(unit 1)
+				)

Commit message: feat: order to JLCPCB
Parts:
- C15: footprint Capacitor_SMD:C_0402_1005Metric -> Capacitor_SMD:C_0603_1608Metric
Changed lines of the file:
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@@
 			)
 		)
-		(property "Footprint" "Capacitor_SMD:C_0402_1005Metric"
+		(property "Footprint" "Capacitor_SMD:C_0603_1608Metric"
 			(at 82.55 90.17 0)
 			(effects
