File: v2.0/main/power.kicad_sch (KiCad schematic)
At the start: 14 parts, among them J5 Battery, Q2 IRLML6402, SW2 EG1215AA, U5 TLV75733PDBV

Commit message: feat: update pcb routing
Parts:
- removed C19: 47u, Capacitor_SMD:C_0603_1608Metric, symbol Device:C_Small
- removed L3: 10u, Inductor_SMD:L_0805_2012Metric, symbol Device:L
- removed R10: 5, Resistor_SMD:R_0805_2012Metric, symbol Device:R_Small
- R7: value 10k -> 6.8k
- R8: value 10k -> 15k
Other:
- moved on the sheet: R8

Commit message: feat: order to JLCPCB
Parts:
- R8: footprint Resistor_SMD:R_0201_0603Metric -> Resistor_SMD:R_0402_1005Metric
- R9: value 1k -> 3.3k
Changed lines of the file:
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@@
 			)
 		)
-		(property "Footprint" "Resistor_SMD:R_0201_0603Metric"
+		(property "Footprint" "Resistor_SMD:R_0402_1005Metric"
 			(at 118.11 102.87 0)
 			(effects
@@
 			)
 		)
-		(property "Value" "1k"
+		(property "Value" "3.3k"
 			(at 201.93 92.7099 0)
 			(effects
