File: v2.0/main/user_interface.kicad_sch (KiCad schematic)
At the start: 26 parts, among them Q3 BSS138, SW3 TVAF06-A020B-R

Commit message: feat: update pcb routing
Parts:
- SP1: footprint omni:STM0440-T-R -> half_mouse_lib:SMT-0440-T-HT-R
- renumbered C21 to C20, D14 to D10, D15 to D11, R13 to R12, R14 to R13, R15 to R14, R16 to R15, R17 to R16, R18 to R17, R19 to R18, R20 to R19, R37 to R20, R38 to R21, R21 to R22, R22 to R23
Changed lines of the file:
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@@
 		(on_board yes)
 		(dnp no)
-		(property "Reference" "C21"
+		(property "Reference" "C20"
 			(at 214.63 105.41 0)
 			(effects
@@
 			(project ""
 				(path "/eb904614-38ff-4497-bc19-593801afccc5/8f985f1a-8d65-4bf2-a1c2-0589d538d088"
-					(reference "C21")
+					(reference "C20")
 					(unit 1)
 				)
@@
 		(on_board yes)
 		(dnp no)
-		(property "Reference" "R21"
+		(property "Reference" "R22"
 			(at 207.2386 90.2716 0)
 			(effects
@@
 			(project ""
 				(path "/eb904614-38ff-4497-bc19-593801afccc5/8f985f1a-8d65-4bf2-a1c2-0589d538d088"
-					(reference "R21")
+					(reference "R22")
 					(unit 1)
 				)
@@
 		(dnp no)
 		(fields_autoplaced yes)
-		(property "Reference" "#PWR050"
+		(property "Reference" "#PWR045"
 			(at 95.25 118.11 0)
 			(effects
@@
 			(project ""
 				(path "/eb904614-38ff-4497-bc19-593801afccc5/8f985f1a-8d65-4bf2-a1c2-0589d538d088"
-					(reference "#PWR050")
+					(reference "#PWR045")
 					(unit 1)
 				)
@@
 		(dnp no)
 		(fields_autoplaced yes)
-		(property "Reference" "R17"
+		(property "Reference" "R16"
 			(at 97.79 96.5199 0)
 			(effects
@@
 			(project ""
 				(path "/eb904614-38ff-4497-bc19-593801afccc5/8f985f1a-8d65-4bf2-a1c2-0589d538d088"
-					(reference "R17")
+					(reference "R16")
 					(unit 1)
 				)
@@
 		(dnp no)
 		(fields_autoplaced yes)
-		(property "Reference" "R13"
+		(property "Reference" "R12"
 			(at 55.88 96.5199 0)
 			(effects
@@
 			(project ""
 				(path "/eb904614-38ff-4497-bc19-593801afccc5/8f985f1a-8d65-4bf2-a1c2-0589d538d088"
-					(reference "R13")
+					(reference "R12")
 					(unit 1)
 				)
@@
 		(dnp no)
 		(fields_autoplaced yes)
-		(property "Reference" "#PWR052"
+		(property "Reference" "#PWR047"
 			(at 115.57 118.11 0)
 			(effects
@@
 			(project ""
 				(path "/eb904614-38ff-4497-bc19-593801afccc5/8f985f1a-8d65-4bf2-a1c2-0589d538d088"
-					(reference "#PWR052")
+					(reference "#PWR047")
 					(unit 1)
 				)
@@
 		(on_board yes)
 		(dnp no)
-		(property "Reference" "#PWR056"
+		(property "Reference" "#PWR053"
 			(at 247.65 91.44 0)
 			(effects
@@
 			(project ""
 				(path "/eb904614-38ff-4497-bc19-593801afccc5/8f985f1a-8d65-4bf2-a1c2-0589d538d088"
-					(reference "#PWR056")
+					(reference "#PWR053")
 					(unit 1)
 				)
@@
 		(on_board yes)
 		(dnp no)
-		(property "Reference" "R22"
+		(property "Reference" "R23"
 			(at 244.2464 104.6734 90)
 			(effects
@@
 			(project ""
 				(path "/eb904614-38ff-4497-bc19-593801afccc5/8f985f1a-8d65-4bf2-a1c2-0589d538d088"
-					(reference "R22")
+					(reference "R23")
 					(unit 1)
 				)
@@
 		(dnp no)
 		(fields_autoplaced yes)
-		(property "Reference" "D14"
+		(property "Reference" "D10"
 			(at 138.43 104.4574 90)
 			(effects
@@
 			(project "main"
 				(path "/eb904614-38ff-4497-bc19-593801afccc5/8f985f1a-8d65-4bf2-a1c2-0589d538d088"
-					(reference "D14")
+					(reference "D10")
 					(unit 1)
 				)
@@
 		(dnp no)
 		(fields_autoplaced yes)
-		(property "Reference" "R37"
+		(property "Reference" "R20"
 			(at 137.16 96.5199 0)
 			(effects
@@
 			(project "main"
 				(path "/eb904614-38ff-4497-bc19-593801afccc5/8f985f1a-8d65-4bf2-a1c2-0589d538d088"
-					(reference "R37")
+					(reference "R20")
 					(unit 1)
 				)
@@
 		(on_board yes)
 		(dnp no)
-		(property "Reference" "#PWR055"
+		(property "Reference" "#PWR052"
 			(at 205.74 118.11 0)
 			(effects
@@
 			(project ""
 				(path "/eb904614-38ff-4497-bc19-593801afccc5/8f985f1a-8d65-4bf2-a1c2-0589d538d088"
-					(reference "#PWR055")
+					(reference "#PWR052")
 					(unit 1)
 				)
@@
 		(dnp no)
 		(fields_autoplaced yes)
-		(property "Reference" "R19"
+		(property "Reference" "R18"
 			(at 118.11 96.5199 0)
 			(effects
@@
 			(project ""
 				(path "/eb904614-38ff-4497-bc19-593801afccc5/8f985f1a-8d65-4bf2-a1c2-0589d538d088"
-					(reference "R19")
+					(reference "R18")
 					(unit 1)
 				)
@@
 		(dnp no)
 		(fields_autoplaced yes)
-		(property "Reference" "R14"
+		(property "Reference" "R13"
 			(at 66.04 96.5199 0)
 			(effects
@@
 			(project ""
 				(path "/eb904614-38ff-4497-bc19-593801afccc5/8f985f1a-8d65-4bf2-a1c2-0589d538d088"
-					(reference "R14")
+					(reference "R13")
 					(unit 1)
 				)
@@
 		(dnp no)
 		(fields_autoplaced yes)
-		(property "Reference" "#PWR051"
+		(property "Reference" "#PWR046"
 			(at 105.41 118.11 0)
 			(effects
@@
 			(project ""
 				(path "/eb904614-38ff-4497-bc19-593801afccc5/8f985f1a-8d65-4bf2-a1c2-0589d538d088"
-					(reference "#PWR051")
+					(reference "#PWR046")
 					(unit 1)
 				)
@@
 		(dnp no)
 		(fields_autoplaced yes)
-		(property "Reference" "R20"
+		(property "Reference" "R19"
 			(at 127 96.5199 0)
 			(effects
@@
 			(project ""
 				(path "/eb904614-38ff-4497-bc19-593801afccc5/8f985f1a-8d65-4bf2-a1c2-0589d538d088"
-					(reference "R20")
+					(reference "R19")
 					(unit 1)
 				)
@@
 		(dnp no)
 		(fields_autoplaced yes)
-		(property "Reference" "R16"
+		(property "Reference" "R15"
 			(at 85.09 96.5199 0)
 			(effects
@@
 			(project ""
 				(path "/eb904614-38ff-4497-bc19-593801afccc5/8f985f1a-8d65-4bf2-a1c2-0589d538d088"
-					(reference "R16")
+					(reference "R15")
 					(unit 1)
 				)
@@
 		(dnp no)
 		(fields_autoplaced yes)
-		(property "Reference" "#PWR073"
+		(property "Reference" "#PWR049"
 			(at 134.62 118.11 0)
 			(effects
@@
 			(project "main"
 				(path "/eb904614-38ff-4497-bc19-593801afccc5/8f985f1a-8d65-4bf2-a1c2-0589d538d088"
-					(reference "#PWR073")
+					(reference "#PWR049")
 					(unit 1)
 				)
@@
 		(dnp no)
 		(fields_autoplaced yes)
-		(property "Reference" "R18"
+		(property "Reference" "R17"
 			(at 107.95 96.5199 0)
 			(effects
@@
 			(project ""
 				(path "/eb904614-38ff-4497-bc19-593801afccc5/8f985f1a-8d65-4bf2-a1c2-0589d538d088"
-					(reference "R18")
+					(reference "R17")
 					(unit 1)
 				)
@@
 		(dnp no)
 		(fields_autoplaced yes)
-		(property "Reference" "#PWR047"
+		(property "Reference" "#PWR042"
 			(at 63.5 118.11 0)
 			(effects
@@
 			(project ""
 				(path "/eb904614-38ff-4497-bc19-593801afccc5/8f985f1a-8d65-4bf2-a1c2-0589d538d088"
-					(reference "#PWR047")
+					(reference "#PWR042")
 					(unit 1)
 				)
@@
 		(dnp no)
 		(fields_autoplaced yes)
-		(property "Reference" "R15"
+		(property "Reference" "R14"
 			(at 76.2 96.5199 0)
 			(effects
@@
 			(project ""
 				(path "/eb904614-38ff-4497-bc19-593801afccc5/8f985f1a-8d65-4bf2-a1c2-0589d538d088"
-					(reference "R15")
+					(reference "R14")
 					(unit 1)
 				)
@@
 		(dnp no)
 		(fields_autoplaced yes)
-		(property "Reference" "#PWR048"
+		(property "Reference" "#PWR043"
 			(at 73.66 118.11 0)
 			(effects
@@
 			(project ""
 				(path "/eb904614-38ff-4497-bc19-593801afccc5/8f985f1a-8d65-4bf2-a1c2-0589d538d088"
-					(reference "#PWR048")
+					(reference "#PWR043")
 					(unit 1)
 				)
@@
 		(dnp no)
 		(fields_autoplaced yes)
-		(property "Reference" "#PWR053"
+		(property "Reference" "#PWR048"
 			(at 124.46 118.11 0)
 			(effects
@@
 			(project ""
 				(path "/eb904614-38ff-4497-bc19-593801afccc5/8f985f1a-8d65-4bf2-a1c2-0589d538d088"
-					(reference "#PWR053")
+					(reference "#PWR048")
 					(unit 1)
 				)
@@
 		(on_board yes)
 		(dnp no)
-		(property "Reference" "#PWR057"
+		(property "Reference" "#PWR054"
 			(at 247.65 118.11 0)
 			(effects
@@
 			(project ""
 				(path "/eb904614-38ff-4497-bc19-593801afccc5/8f985f1a-8d65-4bf2-a1c2-0589d538d088"
-					(reference "#PWR057")
+					(reference "#PWR054")
 					(unit 1)
 				)
@@
 		(dnp no)
 		(fields_autoplaced yes)
-		(property "Reference" "#PWR074"
+		(property "Reference" "#PWR050"
 			(at 143.51 118.11 0)
 			(effects
@@
 			(project "main"
 				(path "/eb904614-38ff-4497-bc19-593801afccc5/8f985f1a-8d65-4bf2-a1c2-0589d538d088"
-					(reference "#PWR074")
+					(reference "#PWR050")
 					(unit 1)
 				)
@@
 		(on_board yes)
 		(dnp no)
-		(property "Reference" "#PWR054"
+		(property "Reference" "#PWR051"
 			(at 205.74 91.44 0)
 			(effects
@@
 			(project ""
 				(path "/eb904614-38ff-4497-bc19-593801afccc5/8f985f1a-8d65-4bf2-a1c2-0589d538d088"
-					(reference "#PWR054")
+					(reference "#PWR051")
 					(unit 1)
 				)
@@
 		(dnp no)
 		(fields_autoplaced yes)
-		(property "Reference" "D15"
+		(property "Reference" "D11"
 			(at 147.32 104.4574 90)
 			(effects
@@
 			(project "main"
 				(path "/eb904614-38ff-4497-bc19-593801afccc5/8f985f1a-8d65-4bf2-a1c2-0589d538d088"
-					(reference "D15")
+					(reference "D11")
 					(unit 1)
 				)
@@
 		(dnp no)
 		(fields_autoplaced yes)
-		(property "Reference" "#PWR049"
+		(property "Reference" "#PWR044"
 			(at 82.55 118.11 0)
 			(effects
@@
 			(project ""
 				(path "/eb904614-38ff-4497-bc19-593801afccc5/8f985f1a-8d65-4bf2-a1c2-0589d538d088"
-					(reference "#PWR049")
+					(reference "#PWR044")
 					(unit 1)
 				)
@@
 		(dnp no)
 		(fields_autoplaced yes)
-		(property "Reference" "R38"
+		(property "Reference" "R21"
 			(at 146.05 96.5199 0)
 			(effects
@@
 			(project "main"
 				(path "/eb904614-38ff-4497-bc19-593801afccc5/8f985f1a-8d65-4bf2-a1c2-0589d538d088"
-					(reference "R38")
+					(reference "R21")
 					(unit 1)
 				)
@@
 		(dnp no)
 		(fields_autoplaced yes)
-		(property "Reference" "#PWR046"
+		(property "Reference" "#PWR041"
 			(at 53.34 118.11 0)
 			(effects
@@
 			(project ""
 				(path "/eb904614-38ff-4497-bc19-593801afccc5/8f985f1a-8d65-4bf2-a1c2-0589d538d088"
-					(reference "#PWR046")
+					(reference "#PWR041")
 					(unit 1)
 				)
@@
 			)
 		)
-		(property "Footprint" "omni:STM0440-T-R"
+		(property "Footprint" "half_mouse_lib:SMT-0440-T-HT-R"
 			(at 256.54 83.82 0)
 			(effects

Commit message: feat: order to JLCPCB
Parts:
- R12, R13, R14, R15, R16, R17, R18, R19, R20, R21: value 1k -> 3.3k
Changed lines of the file:
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@@
 			)
 		)
-		(property "Value" "1k"
+		(property "Value" "3.3k"
 			(at 97.79 99.0599 0)
 			(effects
@@
 			)
 		)
-		(property "Value" "1k"
+		(property "Value" "3.3k"
 			(at 55.88 99.0599 0)
 			(effects
@@
 			)
 		)
-		(property "Value" "1k"
+		(property "Value" "3.3k"
 			(at 137.16 99.0599 0)
 			(effects
@@
 			)
 		)
-		(property "Value" "1k"
+		(property "Value" "3.3k"
 			(at 118.11 99.0599 0)
 			(effects
@@
 			)
 		)
-		(property "Value" "1k"
+		(property "Value" "3.3k"
 			(at 66.04 99.0599 0)
 			(effects
@@
 			)
 		)
-		(property "Value" "1k"
+		(property "Value" "3.3k"
 			(at 127 99.0599 0)
 			(effects
@@
 			)
 		)
-		(property "Value" "1k"
+		(property "Value" "3.3k"
 			(at 85.09 99.0599 0)
 			(effects
@@
 			)
 		)
-		(property "Value" "1k"
+		(property "Value" "3.3k"
 			(at 107.95 99.0599 0)
 			(effects
@@
 			)
 		)
-		(property "Value" "1k"
+		(property "Value" "3.3k"
 			(at 76.2 99.0599 0)
 			(effects
@@
 			)
 		)
-		(property "Value" "1k"
+		(property "Value" "3.3k"
 			(at 146.05 99.0599 0)
 			(effects
